Commit message: update planner

File: niagara_model/urdf/AckermannPlugIn.xacro (robot description, xacro)
@@ -33,5 +33,5 @@
       <!-- output -->
       <publish_odom>true</publish_odom>
-      <publish_odom_tf>false</publish_odom_tf>
+      <publish_odom_tf>true</publish_odom_tf>
       <publish_wheel_tf>true</publish_wheel_tf>
       <publish_distance>false</publish_distance>

File: niagara_model/urdf/DasAutonomeAuto.urdf (robot description, URDF)
Before this commit: robot dasautonomeauto, 3 links, 2 joints
Links:
- removed link test_link
- link base_link: geometry collision mesh filename=file://$(find niagara_model)/meshes/base_link.STL; visual mesh filename=file://$(find niagara_model)/meshes/prius/hybrid_body.obj scale=0.0065 0.0065 0.0065
Joints:
- removed joint base_link_joint_test

File: niagara_model/urdf/VLP-16.xacro (robot description, xacro)
@@ -4,5 +4,5 @@
   <xacro:macro name="VLP-16" params="parent:=base_link name:=velodyne topic:=/velodyne_points hz:=10 lasers:=16 samples:=1875 collision_range:=0.3 min_range:=0.9 max_range:=130.0 noise:=0.008 min_angle:=-${M_PI} max_angle:=${M_PI} gpu:=false">
     <joint name="${name}_base_mount_joint" type="fixed">
-      <origin xyz="0 0 1" rpy="0 0 0" />
+      <origin xyz="-0.2 0 0.8" rpy="0 0 0" />
       <parent link="${parent}"/>
       <child link="${name}_base_link"/>
